File: full_adder_with imput_leds.brd (EAGLE design)
At the start: 100 x 120 mm, 75 parts, among them T101 TPH1R712MD, T102 TPH1R712MD, U1001 FDS6892A, U1002 FDS6892A, U1003 FDS6892A, U101 ATTINY85, U201 CD4052BE, U202 CD4052BE, U203 CD4052BE, U401 KM28C65A-20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

Commit message: drc errors, power planes
Parts:
- added LED1101, LED1102, LED1103, LED1104, LED1105, LED1106, LED1107, LED1108: (no value), led:LED3MM
- added R1101, R1102, R1103, R1104, R1105, R1106, R1107, R1108: 2k2, rcl:R1206
Connections:
- new net N$18: LED1101.A, R1101.1
- new net N$19: LED1102.A, R1102.1
- new net N$20: LED1103.A, R1103.1
- new net N$21: LED1104.A, R1104.1
- new net N$22: LED1105.A, R1105.1
- new net N$23: LED1106.A, R1106.1
- new net N$24: LED1107.A, R1107.1
- new net N$25: LED1108.A, R1108.1
- net A0: now also R1101.2
- net A1: now also R1102.2
- net A2: now also R1103.2
- net A3: now also R1104.2
- net B0: now also R1105.2
- net B1: now also R1106.2
- net B2: now also R1107.2
- net B3: now also R1108.2
- net GND: now also LED1101.K, LED1102.K, LED1103.K, LED1104.K, LED1105.K, LED1106.K, LED1107.K, LED1108.K
Routing:
- net VCC: track 76.3 -> 71.9 mm, vias 7 -> 0
- net N$41: vias 3 -> 2
- removed copper zone on layer 1, net GND
- removed copper zone on layer 16, net N$41
- removed copper zone on layer 16, net VCC
