File: full_adder.sch (EAGLE design)
At the start: 91 parts, among them T101 TPH1R712MD, T102 TPH1R712MD, U1001 FDS6892A, U1002 FDS6892A, U1003 FDS6892A, U101 ATTINY85, U201 CD4052BE, U202 CD4052BE, U203 CD4052BE, U401 KM28C65A-20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

Commit message: drc errors, power planes
Parts:
- removed LED1101, LED1102, LED1103, LED1104, LED1105, LED1106, LED1107, LED1108: (no value), led:LED3MM
- removed R1101, R1102, R1103, R1104, R1105, R1106, R1107, R1108: 2k2, rcl:R-EU_R1206
Connections:
- removed net N$18: LED1101.A, R1101.1
- removed net N$19: LED1102.A, R1102.1
- removed net N$20: LED1103.A, R1103.1
- removed net N$21: LED1104.A, R1104.1
- removed net N$22: LED1105.A, R1105.1
- removed net N$23: LED1106.A, R1106.1
- removed net N$24: LED1107.A, R1107.1
- removed net N$25: LED1108.A, R1108.1
- net A0: no longer R1101.2
- net A1: no longer R1102.2
- net A2: no longer R1103.2
- net A3: no longer R1104.2
- net B0: no longer R1105.2
- net B1: no longer R1106.2
- net B2: no longer R1107.2
- net B3: no longer R1108.2
- net GND: no longer LED1101.C, LED1102.C, LED1103.C, LED1104.C, LED1105.C, LED1106.C, LED1107.C, LED1108.C
Other:
- note removed: "11 Binary Input LEDs"

Commit message: gate resistor
Parts:
- R1001, R1002, R1003, R1004, R1005: value 2k2 -> 10k
- R102: value 100k -> 10k
Other:
- note added: "add 2k2 gate resistor"
Changed lines of the file:
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@@
 <part name="U1001" library="SamacSys_Parts" deviceset="FDS6892A" device=""/>
 <part name="LED1001" library="led" library_urn="urn:adsk.eagle:library:259" deviceset="LED" device="3MM" package3d_urn="urn:adsk.eagle:package:15797/1"/>
-<part name="R1001" library="rcl" library_urn="urn:adsk.eagle:library:334" deviceset="R-EU_" device="R1206" package3d_urn="urn:adsk.eagle:package:23540/2" value="2k2"/>
+<part name="R1001" library="rcl" library_urn="urn:adsk.eagle:library:334" deviceset="R-EU_" device="R1206" package3d_urn="urn:adsk.eagle:package:23540/2" value="10k"/>
 <part name="LED1002" library="led" library_urn="urn:adsk.eagle:library:259" deviceset="LED" device="3MM" package3d_urn="urn:adsk.eagle:package:15797/1"/>
-<part name="R1002" library="rcl" library_urn="urn:adsk.eagle:library:334" deviceset="R-EU_" device="R1206" package3d_urn="urn:adsk.eagle:package:23540/2" value="2k2"/>
+<part name="R1002" library="rcl" library_urn="urn:adsk.eagle:library:334" deviceset="R-EU_" device="R1206" package3d_urn="urn:adsk.eagle:package:23540/2" value="10k"/>
 <part name="LED1003" library="led" library_urn="urn:adsk.eagle:library:259" deviceset="LED" device="3MM" package3d_urn="urn:adsk.eagle:package:15797/1"/>
-<part name="R1003" library="rcl" library_urn="urn:adsk.eagle:library:334" deviceset="R-EU_" device="R1206" package3d_urn="urn:adsk.eagle:package:23540/2" value="2k2"/>
+<part name="R1003" library="rcl" library_urn="urn:adsk.eagle:library:334" deviceset="R-EU_" device="R1206" package3d_urn="urn:adsk.eagle:package:23540/2" value="10k"/>
 <part name="LED1004" library="led" library_urn="urn:adsk.eagle:library:259" deviceset="LED" device="3MM" package3d_urn="urn:adsk.eagle:package:15797/1"/>
-<part name="R1004" library="rcl" library_urn="urn:adsk.eagle:library:334" deviceset="R-EU_" device="R1206" package3d_urn="urn:adsk.eagle:package:23540/2" value="2k2"/>
+<part name="R1004" library="rcl" library_urn="urn:adsk.eagle:library:334" deviceset="R-EU_" device="R1206" package3d_urn="urn:adsk.eagle:package:23540/2" value="10k"/>
 <part name="LED1005" library="led" library_urn="urn:adsk.eagle:library:259" deviceset="LED" device="3MM" package3d_urn="urn:adsk.eagle:package:15797/1"/>
-<part name="R1005" library="rcl" library_urn="urn:adsk.eagle:library:334" deviceset="R-EU_" device="R1206" package3d_urn="urn:adsk.eagle:package:23540/2" value="2k2"/>
+<part name="R1005" library="rcl" library_urn="urn:adsk.eagle:library:334" deviceset="R-EU_" device="R1206" package3d_urn="urn:adsk.eagle:package:23540/2" value="10k"/>
 <part name="GND37" library="supply1" library_urn="urn:adsk.eagle:library:371" deviceset="GND" device=""/>
 <part name="P+23" library="supply1" library_urn="urn:adsk.eagle:library:371" deviceset="VCC" device=""/>
@@
 <part name="R101" library="rcl" library_urn="urn:adsk.eagle:library:334" deviceset="R-EU_" device="R1206" package3d_urn="urn:adsk.eagle:package:23540/2" value="10k"/>
 <part name="GND54" library="supply1" library_urn="urn:adsk.eagle:library:371" deviceset="GND" device=""/>
-<part name="R102" library="rcl" library_urn="urn:adsk.eagle:library:334" deviceset="R-EU_" device="R1206" package3d_urn="urn:adsk.eagle:package:23540/2" value="100k"/>
+<part name="R102" library="rcl" library_urn="urn:adsk.eagle:library:334" deviceset="R-EU_" device="R1206" package3d_urn="urn:adsk.eagle:package:23540/2" value="10k"/>
 <part name="GND47" library="supply1" library_urn="urn:adsk.eagle:library:371" deviceset="GND" device=""/>
 <part name="GND48" library="supply1" library_urn="urn:adsk.eagle:library:371" deviceset="GND" device=""/>
@@
 <wire x1="370.84" y1="175.26" x2="370.84" y2="71.12" width="0.1524" layer="100" style="longdash"/>
 <wire x1="370.84" y1="71.12" x2="370.84" y2="-7.62" width="0.1524" layer="100" style="longdash"/>
+<text x="403.86" y="213.36" size="1.778" layer="91">add 2k2 gate resistor</text>
 </plain>
 <instances>
